File: macropad/macropad.kicad_pcb (KiCad board)
At the start: 2 copper layers, 61 x 42 mm, 7 parts, among them SW1 SW_Push, SW2 SW_Push, SW3 SW_Push, SW4 SW_Push, U1 XIAO-RP2040-DIP

Commit message: Add files via upload
Parts:
- removed D1, D2: SK6812, LED_SMD:LED_SK6812_PLCC4_5.0x5.0mm_P3.2mm
- added LED1: MX_SK6812MINI-E, marbastlib-mx:LED_MX_6028R, B.Cu at (152.3, 90.7)
- added LED2: MX_SK6812MINI-E, marbastlib-mx:LED_MX_6028R, B.Cu at (133.4, 71.8)
- added LED3: MX_SK6812MINI-E, marbastlib-mx:LED_MX_6028R, B.Cu at (114.3, 90.8)
- added LED4: MX_SK6812MINI-E, marbastlib-mx:LED_MX_6028R, B.Cu at (133.3, 90.8)
- moved SW1 0.10 mm to (154.9, 80.6)
Connections:
- U1 pad 13: GND -> Net-(LED1-DIN)
- U1 pad 14: +5V -> Net-(LED1-DOUT)
Routing:
- net Net-(LED1-DOUT): track 0.00 -> 118.9 mm, vias 0 -> 2
- net Net-(LED1-DIN): track 0.00 -> 76.5 mm, vias 0 -> 3
- net Net-(D1-VDD): track 51.4 -> 0.00 mm
- net Net-(LED1-VSS): track 0.00 -> 49.0 mm, vias 0 -> 2
- net +5V: track 45.7 -> 0.00 mm
- net Net-(LED2-VSS): track 0.00 -> 33.1 mm, vias 0 -> 4
- net Net-(LED1-VDD): track 49.5 -> 29.2 mm, vias 1 -> 4
- net GND: track 97.8 -> 80.4 mm
- net Net-(LED3-VSS): track 0.00 -> 14.2 mm
- net Net-(U1-GPIO4/MISO): track 44.3 -> 46.6 mm

Commit message: Add files via upload
Parts:
- added LED5: MX_SK6812MINI-E, marbastlib-mx:LED_MX_6028R, B.Cu at (188.2, 89.9)
- added LED6: MX_SK6812MINI-E, marbastlib-mx:LED_MX_6028R, B.Cu at (149.6, 109.2)
- added LED7: MX_SK6812MINI-E, marbastlib-mx:LED_MX_6028R, B.Cu at (168.9, 109.2)
- added LED8: MX_SK6812MINI-E, marbastlib-mx:LED_MX_6028R, B.Cu at (188.2, 109.3)
- added SW5: SW_Push, Button_Switch_Keyboard:SW_Cherry_MX_1.00u_PCB, F.Cu at (190.8, 79.7)
- added SW6: SW_Push, Button_Switch_Keyboard:SW_Cherry_MX_1.00u_PCB, F.Cu at (152.2, 99.0)
- added SW7: SW_Push, Button_Switch_Keyboard:SW_Cherry_MX_1.00u_PCB, F.Cu at (171.4, 99.1)
- added SW8: SW_Push, Button_Switch_Keyboard:SW_Cherry_MX_1.00u_PCB, F.Cu at (190.8, 99.1)
- U1: moved to F.Cu
- moved LED4 35.6 mm to (168.9, 89.9)
- moved SW4 35.6 mm to (171.4, 79.7)
- moved U1 35.6 mm to (188.5, 64.6), turned to 0 degrees
- moved SW2 35.5 mm to (171.4, 60.4)
- moved LED2 35.5 mm to (168.9, 70.6)
- moved SW3 35.3 mm to (152.2, 79.7)
- moved LED3 35.3 mm to (149.6, 89.9)
- moved SW1 20.4 mm to (152.2, 60.4)
- moved LED1 20.3 mm to (149.6, 70.6)
Connections:
- LED4 pad 4: unconnected-(LED4-VSS-Pad4) -> Net-(LED4-VSS)
- SW1 pad 1: GND -> Net-(LED1-DIN)
- SW2 pad 1: GND -> Net-(LED1-DIN)
- SW3 pad 1: GND -> Net-(LED1-DIN)
- SW4 pad 1: GND -> Net-(LED1-DIN)
- U1 pad 1: unconnected-(U1-GPIO26/ADC0/A0-Pad1) -> Net-(U1-GPIO26/ADC0/A0)
- U1 pad 2: unconnected-(U1-GPIO27/ADC1/A1-Pad2) -> Net-(U1-GPIO27/ADC1/A1)
- U1 pad 3: unconnected-(U1-GPIO28/ADC2/A2-Pad3) -> Net-(U1-GPIO28/ADC2/A2)
- U1 pad 4: unconnected-(U1-GPIO29/ADC3/A3-Pad4) -> Net-(U1-GPIO29/ADC3/A3)
Routing:
- net Net-(U1-GPIO29/ADC3/A3): track 0.00 -> 135.7 mm
- net Net-(U1-GPIO28/ADC2/A2): track 0.00 -> 114.9 mm
- net Net-(LED1-DIN): track 76.5 -> 189.9 mm, vias 3 -> 0
- net Net-(U1-GPIO27/ADC1/A1): track 0.00 -> 94.4 mm
- net Net-(U1-GPIO3/MOSI): track 24.0 -> 112.6 mm, vias 0 -> 2
- net GND: track 80.4 -> 0.00 mm
- net Net-(LED1-DOUT): track 118.9 -> 189.4 mm, vias 2 -> 5
- net Net-(LED5-VSS): track 0.00 -> 58.9 mm, vias 0 -> 2
- net Net-(U1-GPIO1/RX): track 11.2 -> 63.8 mm, vias 0 -> 2
- net Net-(U1-GPIO4/MISO): track 46.6 -> 96.1 mm
- net Net-(U1-GPIO26/ADC0/A0): track 0.00 -> 33.7 mm, vias 0 -> 1
- net Net-(LED1-VSS): track 49.0 -> 15.5 mm
- net Net-(U1-GPIO2/SCK): track 18.6 -> 38.6 mm, vias 0 -> 2
- net Net-(LED6-VSS): track 0.00 -> 15.5 mm, vias 0 -> 2
- net Net-(LED7-VSS): track 0.00 -> 15.4 mm, vias 0 -> 2
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Other:
- board size 61 x 42 mm -> 3.6 x 3.3 mm
- board text added: "AslanPad"
- board text removed: "Aslan's GamePad."
- board text removed: "XIAO HERE"
